Commit message: lidar added

File: description/urdf/robot.urdf.xacro (robot description, xacro)
@@ -3,5 +3,6 @@
     <xacro:include filename="robot_core.xacro"/>
     <xacro:include filename="robot_material.xacro"/>
+    <xacro:include filename="robot_gazebo.xacro"/>
+    <xacro:include filename="robot_lidar.xacro"/>
     <xacro:include filename="inertial_macros.xacro"/>
-    <xacro:include filename="robot_gazebo.xacro"/>
 </robot>

File: description/urdf/robot_core.xacro (robot description, xacro)
@@ -15,4 +15,7 @@
 <xacro:property name="caster_mass" value="0.022"/>
 <xacro:property name="lidar_mass" value="0.207"/>
+<xacro:property name="lidar_radius" value="0.03025"/>
+<xacro:property name="lidar_height" value="0.016"/>
+<xacro:property name="lidar_stand_height" value="0.0424"/>
 <xacro:property name="BLANK" value="0.0"/>
     <!-- BASE LINK -->

File: description/urdf/robot_gazebo.xacro (robot description, xacro)
@@ -34,3 +34,31 @@
         <mu2 value="0.001"/>
     </gazebo>
+    <gazebo reference="laser_frame">
+        <material>Gazebo/Red</material>
+        <sensor name="laser" type="ray">
+            <pose> 0.0 0.0 0.0 0.0 0.0 0.0 </pose>
+            <visualize>true</visualize>
+            <update_rate>10</update_rate>
+            <ray>
+                <scan>
+                    <horizontal>
+                        <samples>360</samples>
+                        <min_angle>-3.14</min_angle>
+                        <max_angle>3.14</max_angle>
+                    </horizontal>
+                </scan>
+                <range>
+                    <min>0.3</min>
+                    <max>12</max>
+                </range>
+            </ray>
+            <plugin name="laser_controller" filename="libgazebo_ros_ray_sensor.so">
+                <ros>
+                    <argument>~/out:=scan</argument>
+                </ros>
+                <output_type>sensor_msgs/LaserScan</output_type>
+                <frame_name>laser_frame</frame_name>
+            </plugin>
+        </sensor>
+    </gazebo>
 </robot>

File: description/urdf/robot_material.xacro (robot description, xacro)
@@ -16,3 +16,6 @@
         <color rgba="0.6 0.6 0.6 1.0"/>
     </material>
+    <material name="red">
+        <color rgba="1 0 0 1"/>
+    </material>
 </robot>
